File: hw/sch_pcb/ISM02A.kicad_sch (KiCad schematic)
At the start: 58 parts, among them J1 JUMP_3X2, J10 HEADER_2x01_PARALLEL, J11 HEADER_2x01_PARALLEL, J12 SMA, J13 U.FL, J14 SMA, J15 U.FL, J16 BMI-S-204-F, J2 SM07B-GHS-TB, J3 HEADER_2x01_PARALLEL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

Commit message: Update title block.
Other:
- company: MLAB www.mlab.cz -> ThunderFly s.r.o.
- title: ISM02A -> TFLORA01A
