File: hw/sch_pcb/TFLORA01B.kicad_pcb (KiCad board)
At the start: 2 copper layers, 50.3 x 30 mm, 55 parts, among them J1 JUMP_3X2, J10 HEADER_2x01_PARALLEL, J11 HEADER_2x01_PARALLEL, J12 MCX, J13 HEADER_2x01_PARALLEL, J15 HEADER_2x01_PARALLEL, J2 HEADER_2x01_PARALLEL, J3 HEADER_2x01_PARALLEL, J4 HEADER_2x01_PARALLEL, J5 HEADER_2x01_PARALLEL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

Commit message: Edit PCB.
Parts:
- removed J11, J13, J15, J2, J4, J5, J6, J7, J8: HEADER_2x01_PARALLEL, Mlab_Pin_Headers:Straight_2x01
- removed M1, M2, M3, M4: HOLE, Mlab_Mechanical:MountingHole_3mm
- removed Y1: 32MHz, Mlab_XTAL:Crystal_SMD_NX2016SA
- added R3: 10k, Resistor_SMD:R_0603_1608Metric, F.Cu at (175.8, 75.2)
- added U4: 74LVC1G157, Package_TO_SOT_SMD:SOT-363_SC-70-6, F.Cu at (173.0, 92.7)
- added X1: IT3205CE 32MHz, Oscillator:Oscillator_DIP-14, F.Cu at (155.1, 84.9)
- C1: value - -> 10pF; footprint Capacitor_SMD:C_0603_1608Metric_Pad1.05x0.95mm_HandSolder -> Capacitor_SMD:C_0603_1608Metric
- C10, C11, C12, C13, C14, C15, C16, C17, C18, C19, C2, C22, C4, C5, C6, C7, C8, C9: footprint Capacitor_SMD:C_0603_1608Metric_Pad1.05x0.95mm_HandSolder -> Capacitor_SMD:C_0603_1608Metric
- C21, C24, C25: footprint Mlab_R:SMD-0805 -> Capacitor_SMD:C_0805_2012Metric
- C3: value - -> 100nF; footprint Capacitor_SMD:C_0603_1608Metric_Pad1.05x0.95mm_HandSolder -> Capacitor_SMD:C_0603_1608Metric; moved to F.Cu
- D1: footprint Mlab_D:Diode-MiniMELF_Standard -> Diode_SMD:D_MiniMELF
- J1: value JUMP_3X2 -> SM07B-GHS-TB; footprint Mlab_Pin_Headers:Straight_2x03 -> Connector_JST:JST_GH_SM07B-GHS-TB_1x07-1MP_P1.25mm_Horizontal
- L1: footprint Mlab_R:SMD-0805 -> Inductor_SMD:L_0805_2012Metric
- R1, R2: footprint Mlab_R:SMD-0603 -> Resistor_SMD:R_0603_1608Metric
- moved C3 44.1 mm to (177.1, 92.0), turned to 0 degrees
- moved J1 16.3 mm to (158.7, 91.9), turned to 0 degrees
Connections:
- C1 pad 2: GND -> Net-(U1-XTA)
- C3 pad 1: Net-(C3-Pad1) -> +3V3
- J1 pad 1: GND -> +5V
- J1 pad 2: GND -> /SCK
- J1 pad 3: +5V -> /MISO
- J1 pad 4: +5V -> /MOSI
- J1 pad 5: GND -> /#CS
- J1 pad 6: GND -> Net-(U4-Y)
- U1 pad 3: Net-(C1-Pad1) -> Net-(U1-XTA)
- U1 pad 4: Net-(C3-Pad1) -> unconnected-(U1-XTB)
- U2 pad 4: (no net) -> unconnected-(U2-NC)
Routing:
- net Net-(U1-XTA): track 0.00 -> 10.8 mm, vias 0 -> 1
- net Net-(C1-Pad1): track 9.53 -> 0.00 mm
- net unconnected-(U1-XTB): track 0.00 -> 8.92 mm
- net Net-(C3-Pad1): track 8.92 -> 0.00 mm
- net GND: track 58.8 -> 57.5 mm, vias 183 -> 182

Commit message: Edit PCB
Parts:
- removed J10, J3, J9: HEADER_2x01_PARALLEL, Mlab_Pin_Headers:Straight_2x01
- added J2: SM03B-GHS-TB, Connector_JST:JST_GH_SM03B-GHS-TB_1x03-1MP_P1.25mm_Horizontal, F.Cu at (139.1, 117.0)
- D1: value BZV55C-5,6V -> BZX585-B5V6.115; footprint Diode_SMD:D_MiniMELF -> Diode_SMD:D_SOD-523
- J1: moved to B.Cu
- J12: footprint Mlab_CON:MCX -> Mlab_CON:MCX_Molex_73415-1061
- moved J1 31.1 mm to (139.5, 116.4), turned to 90 degrees
- moved D1 1.58 mm to (148.1, 108.2), turned to 90 degrees
- turned J12 to 180 degrees
Routing:
- net /#CS: track 30.8 -> 1.67 mm
- net /#RESET: track 30.8 -> 3.04 mm
- net /SCK: track 28.3 -> 1.68 mm
- net /MOSI: track 26.6 -> 0.74 mm
- net /MISO: track 25.5 -> 0.95 mm
- net /DIO2: track 27.0 -> 3.94 mm
- net /BUSY: track 19.6 -> 1.47 mm
- net /DIO1: track 18.4 -> 1.68 mm
- net /DIO3: track 29.1 -> 15.6 mm
- net +3V3: track 65.0 -> 52.2 mm
- net Net-(U1-XTA): track 10.8 -> 1.23 mm
- net Net-(C1-Pad1): track 0.00 -> 9.53 mm
- net +5V: track 18.8 -> 12.9 mm
- net GND: track 57.5 -> 53.4 mm, vias 182 -> 175
