File: hw/sch_pcb/TFLORA01.kicad_sch (KiCad schematic)
At the start: 55 parts, among them J1 SM07B-GHS-TB, J2 MCX, U1 MIC5504-3.3YM5, U2 74LVC1G157, U3 SX1262, U4 PE4259, U5 ECS-TXO-32CSMV-320-AN-TR

Commit message: Improve silkscreen.
Parts:
- C10, C17, C18: MFPN C0G 0,1pF 50V -> (none); UST_ID 5cd09016128750448e45434f -> (none); UST_ID_868 (none) -> 5cd09016128750448e45434f
- C12: UST_ID 5dad549f128750448eca1926 -> (none); UST_ID_868 (none) -> 5dad549f128750448eca1926
- C14: MFPN C0G 0,25pF 50V -> (none); UST_ID 5dad5450128750448eca1919 -> (none); UST_ID_868 (none) -> 5dad5450128750448eca1919
- C15: MFPN C0G 0,1pF 50V -> (none); UST_ID 5c70984812875079b91f8bdd -> (none); UST_ID_868 (none) -> 5c70984812875079b91f8bdd
- C16: MFPN C0G 5% 50V -> (none); UST_ID 5dad549f128750448eca1926 -> (none); UST_ID_868 (none) -> 5dad549f128750448eca1926
- C19: UST_ID 5dad53d8128750448eca1906 -> (none); UST_ID_868 (none) -> 5dad53d8128750448eca1906
- C20: now fitted
- C21: MFPN C0G 0,1pF 50V -> (none); UST_ID 5dad52a4128750448eca18e8 -> (none); UST_ID_868 (none) -> 5dad52a4128750448eca18e8
- L2: UST_ID 5c70984512875079b91f894e -> (none); UST_ID_868 (none) -> 5c70984512875079b91f894e
- L4: UST_ID 671226edd509c19f2ce8ed2d -> (none); UST_ID_868 (none) -> 671226edd509c19f2ce8ed2d
- L5: UST_ID 67122378d509c19f2ce8ecdb -> (none); UST_ID_868 (none) -> 67122378d509c19f2ce8ecdb
- L6: UST_ID 671220a9d509c19f2ce8eca2 -> (none); UST_ID_868 (none) -> 671220a9d509c19f2ce8eca2
Changed lines of the file:
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@@
 			)
 		)
-		(property "UST_ID" "5c70984512875079b91f894e"
+		(property "UST_ID_868" "5c70984512875079b91f894e"
 			(at 218.44 -48.26 0)
 			(effects
@@
 			)
 		)
-		(property "MFPN" "C0G 0,1pF 50V"
-			(at 139.7 87.63 0)
-			(effects
-				(font
-					(size 1.27 1.27)
-				)
-				(hide yes)
-			)
-		)
-		(property "UST_ID" "5cd09016128750448e45434f"
+		(property "UST_ID_868" "5cd09016128750448e45434f"
 			(at 50.8 -76.2 0)
 			(effects
@@
 			)
 		)
+		(property "UST_ID_868" ""
+			(at 133.35 101.6 0)
+			(effects
+				(font
+					(size 1.27 1.27)
+				)
+				(hide yes)
+			)
+		)
+		(property "UST_ID" ""
+			(at 133.35 101.6 0)
+			(effects
+				(font
+					(size 1.27 1.27)
+				)
+				(hide yes)
+			)
+		)
 		(pin "1"
 		)
@@
 			)
 		)
-		(property "MFPN" "C0G 0,25pF 50V"
-			(at 144.78 101.6 0)
-			(effects
-				(font
-					(size 1.27 1.27)
-				)
-				(hide yes)
-			)
-		)
-		(property "UST_ID" "5dad5450128750448eca1919"
+		(property "UST_ID_868" "5dad5450128750448eca1919"
 			(at -24.13 204.47 0)
 			(effects
@@
 			)
 		)
-		(property "UST_ID" "5dad549f128750448eca1926"
+		(property "UST_ID_868" "5dad549f128750448eca1926"
 			(at 53.34 -78.74 0)
+			(effects
+				(font
+					(size 1.27 1.27)
+				)
+				(hide yes)
+			)
+		)
+		(property "UST_ID" ""
+			(at 151.13 96.52 0)
 			(effects
 				(font
@@
 			)
 		)
-		(property "UST_ID" "671226edd509c19f2ce8ed2d"
+		(property "UST_ID_868" "671226edd509c19f2ce8ed2d"
 			(at 257.81 -87.63 0)
 			(effects
@@
 			)
 		)
-		(property "MFPN" "C0G 0,1pF 50V"
-			(at 166.37 101.6 0)
-			(effects
-				(font
-					(size 1.27 1.27)
-				)
-				(hide yes)
-			)
-		)
-		(property "UST_ID" "5c70984812875079b91f8bdd"
+		(property "UST_ID_868" "5c70984812875079b91f8bdd"
 			(at -24.13 204.47 0)
 			(effects
@@
 			)
 		)
-		(property "UST_ID" "671220a9d509c19f2ce8eca2"
+		(property "UST_ID_868" "671220a9d509c19f2ce8eca2"
 			(at 252.73 -1.27 0)
 			(effects
@@
 			)
 		)
-		(property "UST_ID" "5dad53d8128750448eca1906"
+		(property "UST_ID_868" "5dad53d8128750448eca1906"
 			(at -7.62 -17.78 0)
 			(effects
@@
 		(in_bom yes)
 		(on_board yes)
-		(dnp yes)
+		(dnp no)
 		(property "Reference" "C20"
 			(at 136.271 135.9916 0)
@@
 			)
 		)
-		(property "MFPN" "C0G 0,1pF 50V"
-			(at 114.3 148.59 0)
-			(effects
-				(font
-					(size 1.27 1.27)
-				)
-				(hide yes)
-			)
-		)
-		(property "UST_ID" "5dad52a4128750448eca18e8"
+		(property "UST_ID_868" "5dad52a4128750448eca18e8"
 			(at -24.13 298.45 0)
 			(effects
@@
 			)
 		)
-		(property "MFPN" "C0G 5% 50V"
-			(at 214.63 121.92 0)
-			(effects
-				(font
-					(size 1.27 1.27)
-				)
-				(hide yes)
-			)
-		)
-		(property "UST_ID" "5dad549f128750448eca1926"
+		(property "UST_ID_868" "5dad549f128750448eca1926"
 			(at 116.84 -78.74 0)
 			(effects
@@
 			)
 		)
-		(property "MFPN" "C0G 0,1pF 50V"
-			(at 222.25 127 0)
-			(effects
-				(font
-					(size 1.27 1.27)
-				)
-				(hide yes)
-			)
-		)
-		(property "UST_ID" "5cd09016128750448e45434f"
+		(property "UST_ID_868" "5cd09016128750448e45434f"
 			(at 430.53 24.13 0)
 			(effects
@@
 			)
 		)
-		(property "UST_ID" "67122378d509c19f2ce8ecdb"
+		(property "UST_ID_868" "67122378d509c19f2ce8ecdb"
 			(at 327.66 -93.98 0)
 			(effects
@@
 			)
 		)
-		(property "MFPN" "C0G 0,1pF 50V"
-			(at 237.49 127 0)
-			(effects
-				(font
-					(size 1.27 1.27)
-				)
-				(hide yes)
-			)
-		)
-		(property "UST_ID" "5cd09016128750448e45434f"
+		(property "UST_ID_868" "5cd09016128750448e45434f"
 			(at 461.01 24.13 0)
 			(effects
