File: hw/sch_pcb/TFLORA01.kicad_sch (KiCad schematic)
At the start: 55 parts, among them J1 SM07B-GHS-TB, J2 MCX, U1 MIC5504-3.3YM5, U2 74LVC1G157, U3 SX1262, U4 PE4259, U5 ECS-TXO-32CSMV-320-AN-TR

Commit message: Fix kibot warnings.
Parts:
- L6: MFPN LQW18AN15NJ10D -> LQW18AN15NJ10D
Changed lines of the file:
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@@
 			)
 		)
-		(property "UST_id" ""
-			(at 188.595 29.21 0)
-			(effects
-				(font
-					(size 1.27 1.27)
-				)
-				(hide yes)
-			)
-		)
 		(property "UST_ID" "5c70984812875079b91f8bbe"
 			(at -53.975 58.42 0)
@@
 			)
 		)
-		(property "UST_id" ""
-			(at 153.67 29.21 0)
-			(effects
-				(font
-					(size 1.27 1.27)
-				)
-				(hide yes)
-			)
-		)
 		(property "UST_ID" "5c70984812875079b91f8bbe"
 			(at -59.69 59.69 0)
@@
 			)
 		)
-		(property "UST_id" ""
-			(at 120.65 29.21 0)
-			(effects
-				(font
-					(size 1.27 1.27)
-				)
-				(hide yes)
-			)
-		)
 		(property "UST_ID" "5c70984812875079b91f8bbe"
 			(at -59.69 59.69 0)
@@
 			)
 		)
-		(property "MFPN" " LQW18AN15NJ10D"
+		(property "MFPN" "LQW18AN15NJ10D"
 			(at 252.73 -1.27 0)
 			(effects
@@
 			)
 		)
+		(property "UST_ID" ""
+			(at 114.3 137.16 0)
+			(effects
+				(font
+					(size 1.27 1.27)
+				)
+				(hide yes)
+			)
+		)
 		(pin "1"
 		)
@@
 			)
 		)
-		(property "UST_id" ""
-			(at 107.95 29.21 0)
-			(effects
-				(font
-					(size 1.27 1.27)
-				)
-				(hide yes)
-			)
-		)
 		(property "UST_ID" "5cd08b17128750448e4542b1"
 			(at 107.95 29.21 0)
@@
 			)
 		)
-		(property "UST_id" ""
-			(at 203.835 29.21 0)
-			(effects
-				(font
-					(size 1.27 1.27)
-				)
-				(hide yes)
-			)
-		)
 		(property "UST_ID" "60879d38128750769ee58e48"
 			(at 203.835 29.21 0)
@@
 			)
 		)
-		(property "UST_id" ""
-			(at 58.42 142.24 0)
-			(effects
-				(font
-					(size 1.27 1.27)
-				)
-				(hide yes)
-			)
-		)
 		(property "UST_ID" "5c70984412875079b91f8896"
 			(at 58.42 142.24 0)
@@
 			)
 		)
-		(property "UST_id" ""
-			(at 46.99 142.24 0)
-			(effects
-				(font
-					(size 1.27 1.27)
-				)
-				(hide yes)
-			)
-		)
 		(property "UST_ID" "5c70984412875079b91f8896"
 			(at 46.99 142.24 0)
@@
 			(at 107.95 38.1 0)
 			(effects
-				(font
-					(size 1.27 1.27)
-				)
-				(hide yes)
-			)
-		)
-		(property "UST_id" ""
-			(at 107.95 38.1 0)
-			(effects

Commit message: Update submodule.
Parts:
- C4: UST_id C0805_100n -> (none)
Changed lines of the file:
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@@
-			)
-		)
-		(property "UST_id" "C0805_100n"
-			(at 196.215 29.21 0)
-			(effects
-				(font
-					(size 1.27 1.27)
-				)
-				(hide yes)
 			)
 		)
